File: Outdoor_Version/Hardware/AutoGardener_Outdoor.sch (KiCad schematic (older format))
At the start: 26 parts, among them J1 SWO, J2 Header_1x3, J3 Header_1x3, J4 Header_1x2, Q1 FDN308P, Q2 IRLML6346TRPBF, U1 STM32L031K6T6, U2 AP2204RB-3.3TRG1

Commit message: Started a new kicad project.
Parts:
- removed H3: Mounting_hole_unplated_3,2mm, MRS_Mechanical:Mounting_hole_unplated_3,2mm, symbol MRS_Mechanical:Mounting_hole_unplated_3,2mm
Connections:
- net BAT_LO: now also U1.10 (PA4); no longer U1.18 (PA8)
- net OUT1: now also U1.9 (PA3); no longer U1.27 (PB4)
- net SENS_ENA: now also U1.25 (PA15); no longer U1.15 (PB1)
- net UART_RX: now also J2.1; no longer J2.2
- net UART_TX: now also J2.2; no longer J2.1
Changed lines of the file:
@@
 Text Label 10500 1550 2    50   ~ 0
 ADC_SOIL1
-Text Label 8400 2450 0    50   ~ 0
+Text Label 10500 2950 2    50   ~ 0
 SENS_ENA
 Text Label 10500 2450 2    50   ~ 0
@@
 Text Label 10500 2350 2    50   ~ 0
 UART_TX
-Text Label 8400 2650 0    50   ~ 0
+Text Label 10500 1750 2    50   ~ 0
 OUT1
 Wire Wire Line
@@
 Wire Wire Line
 	10500 2550 9950 2550
-Wire Wire Line
-	8950 2450 8400 2450
-Wire Wire Line
-	8950 2650 8400 2650
 Text Label 8800 1950 0    50   ~ 0
 PF0
@@
 	0    -1   -1   0
 $EndComp
-Wire Wire Line
-	10500 2250 9950 2250
-Text Label 10500 2250 2    50   ~ 0
+Text Label 10500 1850 2    50   ~ 0
 BAT_LO
 Text Label 8450 5050 3    50   ~ 0
@@
 $EndComp
 $Comp
-L MRS_Mechanical:Mounting_hole_unplated_3,2mm H3
-U 1 1 5CB0F3CF
-P 10600 4350
-F 0 "H3" H 10600 4450 50  0001 C CNN
-F 1 "Mounting_hole_unplated_3,2mm" H 10600 4250 50  0001 C CNN
-F 2 "MRS_Mechanical:Mounting_hole_unplated_3,2mm" H 10650 4150 50  0001 C CNN
-F 3 "" H 10600 4350 50  0001 C CNN
-	1    10600 4350
-	1    0    0    -1
-$EndComp
-$Comp
 L MRS_MCUs:STM32L031K6T6 U1
 U 1 1 5CAFA03F
@@
 Text Notes 8400 900  0    50   ~ 0
 MCU
+Text Label 8500 3300 0    50   ~ 0
+UART_TX
 Text Label 8500 3200 0    50   ~ 0
-UART_TX
-Text Label 8500 3300 0    50   ~ 0
 UART_RX
 $Comp
@@
 Wire Wire Line
 	8550 1550 8600 1550
+Wire Wire Line
+	10500 1750 9950 1750
+Wire Wire Line
+	10500 1850 9950 1850
+Wire Wire Line
+	10500 2950 9950 2950
 $EndSCHEMATC

Commit message: Finished the design of the outdoor version of the gardener. Generated Gerbers.
Parts:
- removed Q1: FDN308P, MRS_SOT:SOT-23, symbol MRS_Transistors:FDN308P
- removed Q2: IRLML6346TRPBF, MRS_SOT:SOT-23, symbol MRS_Transistors:IRLML6346TRPBF
- removed SB1, SB2: SolderBridge, MRS_Connectors:SB0603, symbol MRS_Connectors:SolderBridge
- added H111: Mr_Gardener_Logo_Small, Logos:mrg_gardener_08mm, symbol Mr_Gardener_Logos:Mr_Gardener_Logo_Small
- added H3, H4, H5, H6: Break_away_tab, MRS_Mechanical:Breakaway_tab_holes, symbol MRS_Mechanical:Break_away_tab
- added Q1, Q2: 2N7002P.215, MRS_SOT:SOT-23, symbol MRS_Transistors:AO3434A
Connections:
- net ADC_SOIL1: now also J3.3; no longer J3.2
- net GND: now also R1.2, U1.31 (BOOT0), Q1.2 (S), Q2.2 (S); no longer J3.3
- net OUT1: now also U1.8 (PA2), Q2.1 (G); no longer R3.1, U1.9 (PA3)
- net SENS_ENA: now also R1.1, Q1.1 (G); no longer R1.2
- net VCC: now also J3.2; no longer R1.1
- net at J4.2: now also Q2.3 (D)
- net VDDA: no longer names the net of J3.1
- net VDDA: now also Q1.3 (D)
- new net LED1: R3.1, U1.9 (PA3)
Other:
- moved on the sheet: R1
Changed lines of the file:
@@
 Text Label 10500 2350 2    50   ~ 0
 UART_TX
-Text Label 10500 1750 2    50   ~ 0
+Text Label 10500 1650 2    50   ~ 0
 OUT1
 Wire Wire Line
@@
 Text Notes 6550 4150 2    50   ~ 0
 3x AAA
-$Comp
-L MRS_Power:VCC #PWR019
-U 1 1 5CACDD15
-P 6550 5650
-F 0 "#PWR019" H 6550 5500 50  0001 C CNN
-F 1 "VCC" H 6567 5823 50  0000 C CNN
-F 2 "" H 6550 5650 50  0001 C CNN
-F 3 "" H 6550 5650 50  0001 C CNN
-	1    6550 5650
-	-1   0    0    -1
-$EndComp
-Text Label 6100 6150 0    50   ~ 0
+Text Label 6150 5850 0    50   ~ 0
 SENS_ENA
 $Comp
 L MRS_Power:GND #PWR046
 U 1 1 5CA0E0BC
-P 7500 5850
-F 0 "#PWR046" H 7500 5600 50  0001 C CNN
-F 1 "GND" H 7505 5677 50  0000 C CNN
-F 2 "" H 7500 5850 50  0001 C CNN
-F 3 "" H 7500 5850 50  0001 C CNN
-	1    7500 5850
-	-1   0    0    -1
-$EndComp
-Text Label 7425 5750 0    50   ~ 0
+P 6850 6150
+F 0 "#PWR046" H 6850 5900 50  0001 C CNN
+F 1 "GND" V 6855 5977 50  0000 C CNN
+F 2 "" H 6850 6150 50  0001 C CNN
+F 3 "" H 6850 6150 50  0001 C CNN
+	1    6850 6150
+	-1   0    0    -1
+$EndComp
+Text Label 7450 5850 0    50   ~ 0
 ADC_SOIL1
-Wire Wire Line
-	7850 5850 7500 5850
-Wire Wire Line
-	7850 5650 7500 5650
 Text Label 9050 5050 3    50   ~ 0
-OUT1
-$Comp
-L MRS_Transistors:IRLML6346TRPBF Q2
-U 1 1 5CAB72CD
-P 10250 5700
-F 0 "Q2" H 10356 5746 50  0000 L CNN
-F 1 "IRLML6346TRPBF" H 10356 5655 50  0000 L CNN
-F 2 "MRS_SOT:SOT-23" H 10250 5375 50  0001 C CNN
-F 3 "https://www.tme.eu/en/Document/4178252f9f9aa1820c70dfb7aab5282b/irlml6346pbf.pdf" H 10250 5450 50  0001 C CNN
-F 4 "IRLML6346TRPBF" H 10250 5300 50  0001 C CNN "TME"
-	1    10250 5700
-	1    0    0    -1
-$EndComp
+LED1
 Wire Wire Line
 	10250 5500 10500 5500
@@
 	10250 5400 10500 5400
 $Comp
-L MRS_Transistors:FDN308P Q1
-U 1 1 5CAFE1A8
-P 6850 5750
-F 0 "Q1" V 7093 5750 50  0000 C CNN
-F 1 "FDN308P" V 7002 5750 50  0000 C CNN
-F 2 "MRS_SOT:SOT-23" H 6850 5400 50  0001 C CNN
-F 3 "https://www.tme.eu/en/Document/dcf621237b7a9c3e175e2f189154a640/FDN308P.pdf" H 6850 5500 50  0001 C CNN
-F 4 "FDN308P" H 6850 5300 50  0001 C CNN "TME"
-	1    6850 5750
-	0    -1   -1   0
-$EndComp
-Wire Wire Line
-	6850 6150 6850 6050
-Wire Wire Line
-	7050 5750 7150 5750
-Wire Wire Line
-	7150 5750 7150 5650
-Wire Wire Line
-	6650 5750 6550 5750
-Wire Wire Line
-	6550 5750 6550 5650
-$Comp
 L MRS_Passives:R R1
 U 1 1 5CB27C07
-P 6550 5950
-F 0 "R1" H 6620 5996 50  0000 L CNN
-F 1 "10k" H 6620 5905 50  0000 L CNN
-F 2 "MRS_Passives:R0603" V 6950 5950 50  0001 C CNN
-F 3 "" V 6630 5950 50  0001 C CNN
-F 4 "WF06P-10K-5%" H 6550 5950 50  0001 C CNN "TME"
-	1    6550 5950
-	1    0    0    -1
-$EndComp
-Wire Wire Line
-	6100 6150 6550 6150
-Wire Wire Line
-	6550 6100 6550 6150
-Connection ~ 6550 6150
-Wire Wire Line
-	6550 6150 6850 6150
-Wire Wire Line
-	6550 5800 6550 5750
-Connection ~ 6550 5750
-$Comp
-L MRS_Power:VDDA #PWR025
-U 1 1 5CAA5030
-P 7150 5650
-F 0 "#PWR025" H 7150 5500 50  0001 C CNN
-F 1 "VDDA" H 7167 5823 50  0000 C CNN
-F 2 "" H 7150 5650 50  0001 C CNN
-F 3 "" H 7150 5650 50  0001 C CNN
-	1    7150 5650
-	1    0    0    -1
-$EndComp
-$Comp
-L MRS_Power:VDDA #PWR049
-U 1 1 5CAA5395
-P 7500 5650
-F 0 "#PWR049" H 7500 5500 50  0001 C CNN
-F 1 "VDDA" H 7517 5823 50  0000 C CNN
-F 2 "" H 7500 5650 50  0001 C CNN
-F 3 "" H 7500 5650 50  0001 C CNN
-	1    7500 5650
+P 6550 6000
+F 0 "R1" H 6620 6046 50  0000 L CNN
+F 1 "10k" H 6620 5955 50  0000 L CNN
+F 2 "MRS_Passives:R0603" V 6950 6000 50  0001 C CNN
+F 3 "" V 6630 6000 50  0001 C CNN
+F 4 "WF06P-10K-5%" H 6550 6000 50  0001 C CNN "TME"
+	1    6550 6000
 	1    0    0    -1
 $EndComp
@@
 PA11
 Wire Wire Line
-	7425 5750 7850 5750
-Wire Wire Line
 	10500 2850 9950 2850
 $Comp
@@
 	1    0    0    -1
 $EndComp
-Wire Wire Line
-	8900 1550 8950 1550
 Text Label 9700 5700 0    50   ~ 0
 OUT1
@@
 Wire Notes Line
 	6050 4800 6050 3700
-$Comp
-L MRS_Connectors:SolderBridge SB2
-U 1 1 5D002CD0
-P 6850 5300
-F 0 "SB2" H 6850 5404 50  0000 C CNN
-F 1 "SolderBridge" H 6850 5200 50  0001 C CNN
-F 2 "MRS_Connectors:SB0603" H 6850 5100 50  0001 C CNN
-F 3 "" H 6850 5300 50  0001 C CNN
-	1    6850 5300
-	1    0    0    -1
-$EndComp
-$Comp
-L MRS_Power:VCC #PWR02
-U 1 1 5D002D80
-P 6550 5300
-F 0 "#PWR02" H 6550 5150 50  0001 C CNN
-F 1 "VCC" H 6567 5473 50  0000 C CNN
-F 2 "" H 6550 5300 50  0001 C CNN
-F 3 "" H 6550 5300 50  0001 C CNN
-	1    6550 5300
-	-1   0    0    -1
-$EndComp
-$Comp
-L MRS_Power:VDDA #PWR05
-U 1 1 5D002DB5
-P 7150 5300
-F 0 "#PWR05" H 7150 5150 50  0001 C CNN
-F 1 "VDDA" H 7167 5473 50  0000 C CNN
-F 2 "" H 7150 5300 50  0001 C CNN
-F 3 "" H 7150 5300 50  0001 C CNN
-	1    7150 5300
-	1    0    0    -1
-$EndComp
-Wire Wire Line
-	7000 5300 7150 5300
-Wire Wire Line
-	6700 5300 6550 5300
 Text Notes 6100 5000 0    50   ~ 0
 Soil moisture measurement
@@
 	1    0    0    -1
 $EndComp
-$Comp
-L MRS_Connectors:SolderBridge SB1
-U 1 1 5D028FCF
-P 8750 1550
-F 0 "SB1" H 8600 1600 50  0000 C CNN
-F 1 "SolderBridge" H 8750 1450 50  0001 C CNN
-F 2 "MRS_Connectors:SB0603" H 8750 1350 50  0001 C CNN
-F 3 "" H 8750 1550 50  0001 C CNN
-	1    8750 1550
-	1    0    0    -1
-$EndComp
 Wire Wire Line
 	8550 1600 8550 1550
 Wire Wire Line
-	8550 1550 8600 1550
-Wire Wire Line
 	10500 1750 9950 1750
 Wire Wire Line
@@
 Wire Wire Line
 	10500 2950 9950 2950
+$Comp
+L Mr_Gardener_Logos:Mr_Gardener_Logo_Small H111
+U 1 1 5D2C678A
+P 8150 3500
+F 0 "H111" H 8150 3650 50  0001 C CNN
+F 1 "Mr_Gardener_Logo_Small" H 8150 3350 50  0001 C CNN
+F 2 "Logos:mrg_gardener_08mm" H 8150 3500 50  0001 C CNN
+F 3 "" H 8150 3500 50  0001 C CNN
+	1    8150 3500
+	1    0    0    -1
+$EndComp
+Wire Wire Line
+	7450 5850 7850 5850
+Wire Wire Line
+	7450 5750 7850 5750
+$Comp
+L MRS_Transistors:AO3434A Q1
+U 1 1 5D2D6490
+P 6850 5850
+F 0 "Q1" H 6956 5896 50  0000 L CNN
+F 1 "2N7002P.215" H 6956 5805 50  0000 L CNN
+F 2 "MRS_SOT:SOT-23" H 6850 5525 50  0001 C CNN
+F 3 "https://www.tme.eu/Document/fda24b70d66290936384ff869f03745e/2N7002P.pdf" H 6850 5600 50  0001 C CNN
+F 4 "2N7002P.215" H 6850 5450 50  0001 C CNN "TME"
+	1    6850 5850
+	1    0    0    -1
+$EndComp
+Wire Wire Line
+	6850 5650 7850 5650
+Wire Wire Line
+	6150 5850 6550 5850
+Connection ~ 6550 5850
+$Comp
+L MRS_Power:GND #PWR0103
+U 1 1 5D2DDD9E
+P 6550 6150
+F 0 "#PWR0103" H 6550 5900 50  0001 C CNN
+F 1 "GND" V 6555 5977 50  0000 C CNN
+F 2 "" H 6550 6150 50  0001 C CNN
+F 3 "" H 6550 6150 50  0001 C CNN
+	1    6550 6150
+	-1   0    0    -1
+$EndComp
+Wire Wire Line
+	6850 6150 6850 6050
+$Comp
+L MRS_Power:VCC #PWR0104
+U 1 1 5D2DF414
+P 7450 5750
+F 0 "#PWR0104" H 7450 5600 50  0001 C CNN
+F 1 "VCC" V 7467 5923 50  0000 C CNN
+F 2 "" H 7450 5750 50  0001 C CNN
+F 3 "" H 7450 5750 50  0001 C CNN
+	1    7450 5750
+	0    -1   -1   0
+$EndComp
+$Comp
+L MRS_Transistors:AO3434A Q2
+U 1 1 5D2DFC92
+P 10250 5700
+F 0 "Q2" H 10356 5746 50  0000 L CNN
+F 1 "2N7002P.215" H 10356 5655 50  0000 L CNN
+F 2 "MRS_SOT:SOT-23" H 10250 5375 50  0001 C CNN
+F 3 "https://www.tme.eu/Document/fda24b70d66290936384ff869f03745e/2N7002P.pdf" H 10250 5450 50  0001 C CNN
+F 4 "2N7002P.215" H 10250 5300 50  0001 C CNN "TME"
+	1    10250 5700
+	1    0    0    -1
+$EndComp
+Wire Wire Line
+	8550 1550 8950 1550
+Text Label 10500 1750 2    50   ~ 0
+LED1
+Wire Wire Line
+	10500 1650 9950 1650
+$Comp
+L MRS_Mechanical:Break_away_tab H6
+U 1 1 5D3F0E44
+P 7500 3550
+F 0 "H6" H 7500 3600 50  0001 C CNN
+F 1 "Break_away_tab" H 7500 3510 50  0001 C CNN
+F 2 "MRS_Mechanical:Breakaway_tab_holes" H 7400 3500 50  0001 C CNN
+F 3 "" H 7500 3550 50  0001 C CNN
+	1    7500 3550
+	1    0    0    -1
+$EndComp
+$Comp
+L MRS_Mechanical:Break_away_tab H5
+U 1 1 5D3F0ED4
+P 7500 3400
+F 0 "H5" H 7500 3450 50  0001 C CNN
+F 1 "Break_away_tab" H 7500 3360 50  0001 C CNN
+F 2 "MRS_Mechanical:Breakaway_tab_holes" H 7400 3350 50  0001 C CNN
+F 3 "" H 7500 3400 50  0001 C CNN
+	1    7500 3400
+	1    0    0    -1
+$EndComp
+$Comp
+L MRS_Mechanical:Break_away_tab H4
+U 1 1 5D3F0F09
+P 7500 3250
+F 0 "H4" H 7500 3300 50  0001 C CNN
+F 1 "Break_away_tab" H 7500 3210 50  0001 C CNN
+F 2 "MRS_Mechanical:Breakaway_tab_holes" H 7400 3200 50  0001 C CNN
+F 3 "" H 7500 3250 50  0001 C CNN
+	1    7500 3250
+	1    0    0    -1
+$EndComp
+$Comp
+L MRS_Mechanical:Break_away_tab H3
+U 1 1 5D3F0F3E
+P 7500 3100
+F 0 "H3" H 7500 3150 50  0001 C CNN
+F 1 "Break_away_tab" H 7500 3060 50  0001 C CNN
+F 2 "MRS_Mechanical:Breakaway_tab_holes" H 7400 3050 50  0001 C CNN
+F 3 "" H 7500 3100 50  0001 C CNN
+	1    7500 3100
+	1    0    0    -1
+$EndComp
 $EndSCHEMATC

Commit message: Added some mechanical details into the PCB document.
Parts:
- removed H3, H4, H5, H6: Break_away_tab, MRS_Mechanical:Breakaway_tab_holes, symbol MRS_Mechanical:Break_away_tab
- BAT1: symbol MRS_Power:Battery -> AutoGardener_Outdoor-rescue:Battery-MRS_Power
- C1, C2, C3, C4, C5, C6, C7: symbol MRS_Passives:C -> AutoGardener_Outdoor-rescue:C-MRS_Passives
- H1, H2: symbol MRS_Mechanical:Mounting_hole_unplated_3,2mm -> AutoGardener_Outdoor-rescue:Mounting_hole_unplated_3,2mm-MRS_Mechanical
- H111: symbol Mr_Gardener_Logos:Mr_Gardener_Logo_Small -> AutoGardener_Outdoor-rescue:Mr_Gardener_Logo_Small-Mr_Gardener_Logos
- J1: symbol MRS_Connectors:Header_1x5 -> AutoGardener_Outdoor-rescue:Header_1x5-MRS_Connectors
- J2, J3: symbol MRS_Connectors:Header_1x3 -> AutoGardener_Outdoor-rescue:Header_1x3-MRS_Connectors
- J4: symbol MRS_Connectors:Header_1x2 -> AutoGardener_Outdoor-rescue:Header_1x2-MRS_Connectors
- LD13, LD3: symbol MRS_Diodes:Diode_LED_0805 -> AutoGardener_Outdoor-rescue:Diode_LED_0805-MRS_Diodes
- Q1, Q2: symbol MRS_Transistors:AO3434A -> AutoGardener_Outdoor-rescue:AO3434A-MRS_Transistors
- R1, R2, R3: symbol MRS_Passives:R -> AutoGardener_Outdoor-rescue:R-MRS_Passives
- U1: symbol MRS_MCUs:STM32L031K6T6 -> AutoGardener_Outdoor-rescue:STM32L031K6T6-MRS_MCUs
- U2: symbol MRS_Power_Management:AP2204RB-3.3TRG1 -> AutoGardener_Outdoor-rescue:AP2204RB-3.3TRG1-MRS_Power_Management
Changed lines of the file:
@@
 NoConn ~ 8800 1950
 $Comp
-L MRS_Power:VCC #PWR012
+L AutoGardener_Outdoor-rescue:VCC-MRS_Power #PWR012
 U 1 1 5CA00ECE
 P 9450 1050
@@
 	9550 1150 9550 1250
 $Comp
-L MRS_Power:GND #PWR010
+L AutoGardener_Outdoor-rescue:GND-MRS_Power #PWR010
 U 1 1 5CA02368
 P 9400 3350
@@
 Connection ~ 9400 3250
 $Comp
-L MRS_Diodes:Diode_LED_0805 LD3
+L AutoGardener_Outdoor-rescue:Diode_LED_0805-MRS_Diodes LD3
 U 1 1 5CA03BD4
 P 9050 5750
@@
 $EndComp
 $Comp
-L MRS_Diodes:Diode_LED_0805 LD13
+L AutoGardener_Outdoor-rescue:Diode_LED_0805-MRS_Diodes LD13
 U 1 1 5CA03D99
 P 8450 5800
@@
 BAT_LO
 $Comp
-L MRS_Power:GND #PWR055
+L AutoGardener_Outdoor-rescue:GND-MRS_Power #PWR055
 U 1 1 5CA0A3CD
 P 9050 6000
@@
 $EndComp
 $Comp
-L MRS_Power:GND #PWR022
+L AutoGardener_Outdoor-rescue:GND-MRS_Power #PWR022
 U 1 1 5CA0A462
 P 8450 6050
@@
 	8450 5950 8450 6050
 $Comp
-L MRS_Passives:R R3
+L AutoGardener_Outdoor-rescue:R-MRS_Passives R3
 U 1 1 5CA0E06E
 P 9050 5450
@@
 $EndComp
 $Comp
-L MRS_Passives:R R2
+L AutoGardener_Outdoor-rescue:R-MRS_Passives R2
 U 1 1 5CA0E18A
 P 8450 5500
@@
 BAT LOW
 $Comp
-L MRS_Passives:C C1
+L AutoGardener_Outdoor-rescue:C-MRS_Passives C1
 U 1 1 5CA1A1FA
 P 10900 1600
@@
 $EndComp
 $Comp
-L MRS_Power:VCC #PWR013
+L AutoGardener_Outdoor-rescue:VCC-MRS_Power #PWR013
 U 1 1 5CA1A310
 P 10900 1450
@@
 $EndComp
 $Comp
-L MRS_Power:GND #PWR014
+L AutoGardener_Outdoor-rescue:GND-MRS_Power #PWR014
 U 1 1 5CA1A337
 P 10900 1750
@@
 $EndComp
 $Comp
-L MRS_Passives:C C2
+L AutoGardener_Outdoor-rescue:C-MRS_Passives C2
 U 1 1 5CA1AEDD
 P 10900 2350
@@
 $EndComp
 $Comp
-L MRS_Power:VCC #PWR016
+L AutoGardener_Outdoor-rescue:VCC-MRS_Power #PWR016
 U 1 1 5CA1AEE4
 P 10900 2200
@@
 $EndComp
 $Comp
-L MRS_Power:GND #PWR017
+L AutoGardener_Outdoor-rescue:GND-MRS_Power #PWR017
 U 1 1 5CA1AEEA
 P 10900 2500
@@
 $EndComp
 $Comp
-L MRS_Passives:C C3
+L AutoGardener_Outdoor-rescue:C-MRS_Passives C3
 U 1 1 5CA1BA39
 P 10900 3100
@@
 $EndComp
 $Comp
-L MRS_Power:VCC #PWR020
+L AutoGardener_Outdoor-rescue:VCC-MRS_Power #PWR020
 U 1 1 5CA1BA40
 P 10900 2950
@@
 $EndComp
 $Comp
-L MRS_Power:GND #PWR021
+L AutoGardener_Outdoor-rescue:GND-MRS_Power #PWR021
 U 1 1 5CA1BA46
 P 10900 3250
@@
 VDDIO
 $Comp
-L MRS_Passives:C C5
+L AutoGardener_Outdoor-rescue:C-MRS_Passives C5
 U 1 1 5CA26949
 P 7200 4250
@@
 $EndComp
 $Comp
-L MRS_Passives:C C4
+L AutoGardener_Outdoor-rescue:C-MRS_Passives C4
 U 1 1 5CA26A1F
 P 6800 4250
@@
 $EndComp
 $Comp
-L MRS_Power:GND #PWR09
+L AutoGardener_Outdoor-rescue:GND-MRS_Power #PWR09
 U 1 1 5CA30E44
 P 6800 4400
@@
 $EndComp
 $Comp
-L MRS_Power:GND #PWR011
+L AutoGardener_Outdoor-rescue:GND-MRS_Power #PWR011
 U 1 1 5CA32305
 P 7200 4400
@@
 3V3
 $Comp
-L MRS_Power:GND #PWR015
+L AutoGardener_Outdoor-rescue:GND-MRS_Power #PWR015
 U 1 1 5CA3D650
 P 7850 4400
@@
 $EndComp
 $Comp
-L MRS_Power:Battery BAT1
+L AutoGardener_Outdoor-rescue:Battery-MRS_Power BAT1
 U 1 1 5CA6EBCF
 P 6200 4250
@@
 $EndComp
 $Comp
-L MRS_Power:GND #PWR04
+L AutoGardener_Outdoor-rescue:GND-MRS_Power #PWR04
 U 1 1 5CA6ECC3
 P 6200 4450
@@
 SENS_ENA
 $Comp
-L MRS_Power:GND #PWR046
+L AutoGardener_Outdoor-rescue:GND-MRS_Power #PWR046
 U 1 1 5CA0E0BC
 P 6850 6150
@@
 	10250 5500 10500 5500
 $Comp
-L MRS_Power:GND #PWR066
+L AutoGardener_Outdoor-rescue:GND-MRS_Power #PWR066
 U 1 1 5CAB72D5
 P 10250 5900
@@
 	10250 5400 10500 5400
 $Comp
-L MRS_Passives:R R1
+L AutoGardener_Outdoor-rescue:R-MRS_Passives R1
 U 1 1 5CB27C07
 P 6550 6000
@@
 $EndComp
 $Comp
-L MRS_Power:VCC #PWR0101
+L AutoGardener_Outdoor-rescue:VCC-MRS_Power #PWR0101
 U 1 1 5CAA5D7D
 P 9350 4100
@@
 $EndComp
 $Comp
-L MRS_Power:GND #PWR0102
+L AutoGardener_Outdoor-rescue:GND-MRS_Power #PWR0102
 U 1 1 5CAA66D8
 P 9350 4500
@@
 	9550 4300 9850 4300
 $Comp
-L MRS_Connectors:Header_1x5 J1
+L AutoGardener_Outdoor-rescue:Header_1x5-MRS_Connectors J1
 U 1 1 5CAE6D61
 P 10000 4250
@@
 $EndComp
 $Comp
-L MRS_Mechanical:Mounting_hole_unplated_3,2mm H1
+L AutoGardener_Outdoor-rescue:Mounting_hole_unplated_3,2mm-MRS_Mechanical H1
 U 1 1 5CB29AA5
 P 10600 4050
@@
 $EndComp
 $Comp
-L MRS_Power_Management:AP2204RB-3.3TRG1 U2
+L AutoGardener_Outdoor-rescue:AP2204RB-3.3TRG1-MRS_Power_Management U2
 U 1 1 5CAD38B8
 P 7850 4100
@@
 $EndComp
 $Comp
-L MRS_Passives:C C6
+L AutoGardener_Outdoor-rescue:C-MRS_Passives C6
 U 1 1 5CAD3977
 P 8350 4250
@@
 $EndComp
 $Comp
-L MRS_Passives:C C7
+L AutoGardener_Outdoor-rescue:C-MRS_Passives C7
 U 1 1 5CAD3BF7
 P 8800 4250
@@
 	8350 4100 8800 4100
 $Comp
-L MRS_Power:GND #PWR0105
+L AutoGardener_Outdoor-rescue:GND-MRS_Power #PWR0105
 U 1 1 5CAF04F3
 P 8350 4400
@@
 $EndComp
 $Comp
-L MRS_Power:GND #PWR0106
+L AutoGardener_Outdoor-rescue:GND-MRS_Power #PWR0106
 U 1 1 5CAF057C
 P 8800 4400
@@
 Connection ~ 8350 4100
 $Comp
-L MRS_Mechanical:Mounting_hole_unplated_3,2mm H2
+L AutoGardener_Outdoor-rescue:Mounting_hole_unplated_3,2mm-MRS_Mechanical H2
 U 1 1 5CB07C28
 P 10600 4200
@@
 $EndComp
 $Comp
-L MRS_MCUs:STM32L031K6T6 U1
+L AutoGardener_Outdoor-rescue:STM32L031K6T6-MRS_MCUs U1
 U 1 1 5CAFA03F
 P 9450 2250
@@
 	10500 2850 9950 2850
 $Comp
-L MRS_Power:VCC #PWR0107
+L AutoGardener_Outdoor-rescue:VCC-MRS_Power #PWR0107
 U 1 1 5CB44371
 P 10500 1450
@@
 $EndComp
 $Comp
-L MRS_Power:GND #PWR07
+L AutoGardener_Outdoor-rescue:GND-MRS_Power #PWR07
 U 1 1 5CDAEFB6
 P 8550 1600
@@
 	9700 5700 9950 5700
 $Comp
-L MRS_Power:+5V #PWR03
+L AutoGardener_Outdoor-rescue:+5V-MRS_Power #PWR03
 U 1 1 5CFF4583
 P 6800 4100
@@
 Connection ~ 6800 4100
 $Comp
-L MRS_Power:+5V #PWR01
+L AutoGardener_Outdoor-rescue:+5V-MRS_Power #PWR01
 U 1 1 5CFF45E4
 P 6200 4050
@@
 Connection ~ 8800 4100
 $Comp
-L MRS_Power:VCC #PWR037
+L AutoGardener_Outdoor-rescue:VCC-MRS_Power #PWR037
 U 1 1 5CA3D277
 P 8800 4100
@@
 	9550 4900 8250 4900
 $Comp
-L MRS_Power:+5V #PWR08
+L AutoGardener_Outdoor-rescue:+5V-MRS_Power #PWR08
 U 1 1 5D008108
 P 10250 5300
@@
 UART_RX
 $Comp
-L MRS_Power:GND #PWR06
+L AutoGardener_Outdoor-rescue:GND-MRS_Power #PWR06
 U 1 1 5D022E97
 P 8800 3400
@@
 	8500 3200 8900 3200
 $Comp
-L MRS_Connectors:Header_1x3 J3
+L AutoGardener_Outdoor-rescue:Header_1x3-MRS_Connectors J3
 U 1 1 5D0282F4
 P 8000 5700
@@
 $EndComp
 $Comp
-L MRS_Connectors:Header_1x2 J4
+L AutoGardener_Outdoor-rescue:Header_1x2-MRS_Connectors J4
 U 1 1 5D028386
 P 10650 5450
@@
 $EndComp
 $Comp
-L MRS_Connectors:Header_1x3 J2
+L AutoGardener_Outdoor-rescue:Header_1x3-MRS_Connectors J2
 U 1 1 5D0289F1
 P 9050 3250
@@
 	10500 2950 9950 2950
 $Comp
-L Mr_Gardener_Logos:Mr_Gardener_Logo_Small H111
+L AutoGardener_Outdoor-rescue:Mr_Gardener_Logo_Small-Mr_Gardener_Logos H111
 U 1 1 5D2C678A
 P 8150 3500
@@
 	7450 5750 7850 5750
 $Comp
-L MRS_Transistors:AO3434A Q1
+L AutoGardener_Outdoor-rescue:AO3434A-MRS_Transistors Q1
 U 1 1 5D2D6490
 P 6850 5850
@@
 Connection ~ 6550 5850
 $Comp
-L MRS_Power:GND #PWR0103
+L AutoGardener_Outdoor-rescue:GND-MRS_Power #PWR0103
 U 1 1 5D2DDD9E
 P 6550 6150
@@
 	6850 6150 6850 6050
 $Comp
-L MRS_Power:VCC #PWR0104
+L AutoGardener_Outdoor-rescue:VCC-MRS_Power #PWR0104
 U 1 1 5D2DF414
 P 7450 5750
@@
 $EndComp
 $Comp
-L MRS_Transistors:AO3434A Q2
+L AutoGardener_Outdoor-rescue:AO3434A-MRS_Transistors Q2
 U 1 1 5D2DFC92
 P 10250 5700
@@
 Wire Wire Line
 	10500 1650 9950 1650
-$Comp
-L MRS_Mechanical:Break_away_tab H6
-U 1 1 5D3F0E44
-P 7500 3550
-F 0 "H6" H 7500 3600 50  0001 C CNN
-F 1 "Break_away_tab" H 7500 3510 50  0001 C CNN
-F 2 "MRS_Mechanical:Breakaway_tab_holes" H 7400 3500 50  0001 C CNN
-F 3 "" H 7500 3550 50  0001 C CNN
-	1    7500 3550
-	1    0    0    -1
-$EndComp
-$Comp
-L MRS_Mechanical:Break_away_tab H5
-U 1 1 5D3F0ED4
-P 7500 3400
-F 0 "H5" H 7500 3450 50  0001 C CNN
-F 1 "Break_away_tab" H 7500 3360 50  0001 C CNN
-F 2 "MRS_Mechanical:Breakaway_tab_holes" H 7400 3350 50  0001 C CNN
-F 3 "" H 7500 3400 50  0001 C CNN
-	1    7500 3400
-	1    0    0    -1
-$EndComp
-$Comp
-L MRS_Mechanical:Break_away_tab H4
-U 1 1 5D3F0F09
-P 7500 3250
-F 0 "H4" H 7500 3300 50  0001 C CNN
-F 1 "Break_away_tab" H 7500 3210 50  0001 C CNN
-F 2 "MRS_Mechanical:Breakaway_tab_holes" H 7400 3200 50  0001 C CNN
-F 3 "" H 7500 3250 50  0001 C CNN
-	1    7500 3250
-	1    0    0    -1
-$EndComp
-$Comp
-L MRS_Mechanical:Break_away_tab H3
-U 1 1 5D3F0F3E
-P 7500 3100
-F 0 "H3" H 7500 3150 50  0001 C CNN
-F 1 "Break_away_tab" H 7500 3060 50  0001 C CNN
-F 2 "MRS_Mechanical:Breakaway_tab_holes" H 7400 3050 50  0001 C CNN
-F 3 "" H 7500 3100 50  0001 C CNN
-	1    7500 3100
-	1    0    0    -1
-$EndComp
 $EndSCHEMATC
