File: Indoor_Version/Hardware/Plant_monitoring_device.sch (KiCad schematic (older format))
At the start: 74 parts, among them J1 Barrel_Jack, J10 A2501WR-2P1, J11 S3B-ZR, J12 S3B-ZR, J13 S3B-ZR, J14 S3B-ZR, J15 S2B-ZR, J2 Header_1x6, J3 A2501WR-2P1, J4 A2501WR-2P1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

Commit message: Merging.
Parts:
- C21, C31, C33: TME CL10A106MO8NQNC -> CL32B106KAJNNNE
- J10, J3, J4, J5, J6, J7, J8, J9: TME NXW-02K, NXG-02, NXG-T -> NX2500-02SMR
- R111, R112, R113: TME (none) -> WF06P-150R-5%
- R32: TME WF06P-10K-5% -> CQ0603-49K9-1%
- R33: TME WF06P-10K-5% -> SMD0603-16K
- U1: TME (none) -> ESP32-WROOM-32D
Changed lines of the file:
@@
 F 2 "MRS_Passives:C1210" H 2200 1000 50  0001 C CNN
 F 3 "" H 2225 1600 50  0001 C CNN
-F 4 "CL10A106MO8NQNC" H 2200 1500 50  0001 C CNN "TME"
+F 4 "CL32B106KAJNNNE" H 2200 1500 50  0001 C CNN "TME"
 	1    2200 1500
 	1    0    0    -1
@@
 F 2 "MRS_Passives:C1210" H 5150 1000 50  0001 C CNN
 F 3 "" H 5175 1600 50  0001 C CNN
-F 4 "CL10A106MO8NQNC" H 5150 1500 50  0001 C CNN "TME"
+F 4 "CL32B106KAJNNNE" H 5150 1500 50  0001 C CNN "TME"
 	1    5150 1500
 	1    0    0    -1
@@
 F 2 "MRS_Connectors:A2501WR-2P1" H 8600 650 50  0001 C CNN
 F 3 "https://www.tme.eu/Document/cd32a27eaa56cbe24bba92418ea31066/A2501WR-XP.pdf" H 8600 550 50  0001 C CNN
-F 4 "NXW-02K, NXG-02, NXG-T" H 8600 450 50  0001 C CNN "TME"
+F 4 "NX2500-02SMR" H 8600 450 50  0001 C CNN "TME"
 	1    8600 900
 	1    0    0    -1
@@
 F 2 "MRS_Connectors:A2501WR-2P1" H 8600 1750 50  0001 C CNN
 F 3 "https://www.tme.eu/Document/cd32a27eaa56cbe24bba92418ea31066/A2501WR-XP.pdf" H 8600 1650 50  0001 C CNN
-F 4 "NXW-02K, NXG-02, NXG-T" H 8600 1550 50  0001 C CNN "TME"
+F 4 "NX2500-02SMR" H 8600 1550 50  0001 C CNN "TME"
 	1    8600 2000
 	1    0    0    -1
@@
 F 2 "MRS_Connectors:A2501WR-2P1" H 8600 2850 50  0001 C CNN
 F 3 "https://www.tme.eu/Document/cd32a27eaa56cbe24bba92418ea31066/A2501WR-XP.pdf" H 8600 2750 50  0001 C CNN
-F 4 "NXW-02K, NXG-02, NXG-T" H 8600 2650 50  0001 C CNN "TME"
+F 4 "NX2500-02SMR" H 8600 2650 50  0001 C CNN "TME"
 	1    8600 3100
 	1    0    0    -1
@@
 F 2 "MRS_Connectors:A2501WR-2P1" H 8600 3950 50  0001 C CNN
 F 3 "https://www.tme.eu/Document/cd32a27eaa56cbe24bba92418ea31066/A2501WR-XP.pdf" H 8600 3850 50  0001 C CNN
-F 4 "NXW-02K, NXG-02, NXG-T" H 8600 3750 50  0001 C CNN "TME"
+F 4 "NX2500-02SMR" H 8600 3750 50  0001 C CNN "TME"
 	1    8600 4200
 	1    0    0    -1
@@
 F 2 "MRS_Connectors:A2501WR-2P1" H 10600 650 50  0001 C CNN
 F 3 "https://www.tme.eu/Document/cd32a27eaa56cbe24bba92418ea31066/A2501WR-XP.pdf" H 10600 550 50  0001 C CNN
-F 4 "NXW-02K, NXG-02, NXG-T" H 10600 450 50  0001 C CNN "TME"
+F 4 "NX2500-02SMR" H 10600 450 50  0001 C CNN "TME"
 	1    10600 900
 	1    0    0    -1
@@
 F 2 "MRS_Connectors:A2501WR-2P1" H 10600 1750 50  0001 C CNN
 F 3 "https://www.tme.eu/Document/cd32a27eaa56cbe24bba92418ea31066/A2501WR-XP.pdf" H 10600 1650 50  0001 C CNN
-F 4 "NXW-02K, NXG-02, NXG-T" H 10600 1550 50  0001 C CNN "TME"
+F 4 "NX2500-02SMR" H 10600 1550 50  0001 C CNN "TME"
 	1    10600 2000
 	1    0    0    -1
@@
 F 2 "MRS_Connectors:A2501WR-2P1" H 10600 2850 50  0001 C CNN
 F 3 "https://www.tme.eu/Document/cd32a27eaa56cbe24bba92418ea31066/A2501WR-XP.pdf" H 10600 2750 50  0001 C CNN
-F 4 "NXW-02K, NXG-02, NXG-T" H 10600 2650 50  0001 C CNN "TME"
+F 4 "NX2500-02SMR" H 10600 2650 50  0001 C CNN "TME"
 	1    10600 3100
 	1    0    0    -1
@@
 F 2 "MRS_Connectors:A2501WR-2P1" H 10600 3950 50  0001 C CNN
 F 3 "https://www.tme.eu/Document/cd32a27eaa56cbe24bba92418ea31066/A2501WR-XP.pdf" H 10600 3850 50  0001 C CNN
-F 4 "NXW-02K, NXG-02, NXG-T" H 10600 3750 50  0001 C CNN "TME"
+F 4 "NX2500-02SMR" H 10600 3750 50  0001 C CNN "TME"
 	1    10600 4200
 	1    0    0    -1
@@
 F 2 "MRS_Communication:ESP32-WROOM" H 2650 4700 50  0001 C CNN
 F 3 "https://www.espressif.com/sites/default/files/documentation/esp32-wroom-32_datasheet_en.pdf" H 2650 4600 50  0001 C CNN
+F 4 "ESP32-WROOM-32D" H 0   0   50  0001 C CNN "TME"
 	1    2650 5800
 	1    0    0    -1
@@
 F 2 "MRS_Passives:R0603" V 5150 1350 50  0001 C CNN
 F 3 "" V 4830 1350 50  0001 C CNN
-F 4 "WF06P-10K-5%" H 4750 1350 50  0001 C CNN "TME"
+F 4 "CQ0603-49K9-1%" H 4750 1350 50  0001 C CNN "TME"
 	1    4750 1350
 	1    0    0    -1
@@
 F 2 "MRS_Passives:R0603" V 5150 1650 50  0001 C CNN
 F 3 "" V 4830 1650 50  0001 C CNN
-F 4 "WF06P-10K-5%" H 4750 1650 50  0001 C CNN "TME"
+F 4 "SMD0603-16K" H 4750 1650 50  0001 C CNN "TME"
 	1    4750 1650
 	1    0    0    -1
@@
 F 2 "MRS_Passives:C1210" H 800 2600 50  0001 C CNN
 F 3 "" H 825 3200 50  0001 C CNN
-F 4 "CL10A106MO8NQNC" H 800 3100 50  0001 C CNN "TME"
+F 4 "CL32B106KAJNNNE" H 800 3100 50  0001 C CNN "TME"
 	1    800  3100
 	1    0    0    -1
@@
 F 2 "MRS_Passives:R0603" V 6300 6950 50  0001 C CNN
 F 3 "" V 5980 6950 50  0001 C CNN
+F 4 "WF06P-150R-5%" H 0   0   50  0001 C CNN "TME"
 	1    5900 6950
 	0    1    1    0
@@
 F 2 "MRS_Passives:R0603" V 6300 7350 50  0001 C CNN
 F 3 "" V 5980 7350 50  0001 C CNN
+F 4 "WF06P-150R-5%" H 0   0   50  0001 C CNN "TME"
 	1    5900 7350
 	0    1    1    0
@@
 F 2 "MRS_Passives:R0603" V 6300 7150 50  0001 C CNN
 F 3 "" V 5980 7150 50  0001 C CNN
+F 4 "WF06P-150R-5%" H 0   0   50  0001 C CNN "TME"
 	1    5900 7150
 	0    1    1    0
